Commit message: [UPD] ros2 style sdf

File: tmc_wrs_gazebo_worlds/worlds/include/physics.xacro (robot description, xacro)
@@ -1,3 +1,3 @@
-<?xml version="1.0" ?>
+<?xml version="1.0" encoding="UTF-8" ?>
 <!--
 Copyright (c) 2017, Toyota Motor Corporation
@@ -25,29 +25,79 @@
 POSSIBILITY OF SUCH DAMAGE.
 -->
-<sdf version="1.4" xmlns:xacro="http://www.ros.org/wiki/xacro">
-  <xacro:arg name="fast_physics" default="true" />
-  <xacro:arg name="highrtf" default="false" />
-  <physics type="ode">
-    <xacro:if value="$(arg fast_physics)">
-    <xacro:unless value="$(arg highrtf)">
-    <real_time_update_rate>333.0</real_time_update_rate>
-    </xacro:unless>
-    <xacro:if value="$(arg highrtf)">
-    <real_time_update_rate>0</real_time_update_rate>
-    </xacro:if>
-    <max_step_size>0.003</max_step_size>
-    <ode>
-      <solver>
-        <type>quick</type>
-        <iters>100</iters>
-      </solver>
-      <constraints>
-        <cfm>0.0001</cfm>
-      </constraints>
-    </ode>
-    </xacro:if>
-    <xacro:if value="$(arg highrtf)">
-    <real_time_update_rate>0</real_time_update_rate>
-    </xacro:if>
-  </physics>
+<sdf version="1.8" xmlns:xacro="http://www.ros.org/wiki/xacro">
+  <xacro:macro name="physics" params="fast_physics:=true highrtf:=false" >
+    <physics name="1ms" type="ignored">
+      <xacro:if value="$(arg fast_physics)">
+        <xacro:unless value="$(arg highrtf)">
+          <real_time_update_rate>333.0</real_time_update_rate>
+        </xacro:unless>
+        <xacro:if value="$(arg highrtf)">
+          <real_time_update_rate>0</real_time_update_rate>
+        </xacro:if>
+        <max_step_size>0.003</max_step_size>
+      </xacro:if>
+      <xacro:if value="$(arg highrtf)">
+        <real_time_update_rate>0</real_time_update_rate>
+      </xacro:if>
+    </physics>
+    <plugin name='gz::sim::systems::Physics' filename='gz-sim-physics-system'/>
+    <plugin name='gz::sim::systems::UserCommands' filename='gz-sim-user-commands-system'/>
+    <plugin name='gz::sim::systems::SceneBroadcaster' filename='gz-sim-scene-broadcaster-system'/>
+    <!-- <plugin name='gz::sim::systems::Contact' filename='gz-sim-contact-system'/> -->
+    <!-- <plugin name='gz::sim::systems::Imu' filename='gz-sim-imu-system'/> -->
+    <!-- <plugin name='gz::sim::systems::AirPressure' filename='gz-sim-air-pressure-system'/> -->
+    <!-- <plugin name='gz::sim::systems::ApplyLinkWrench' filename='gz-sim-apply-link-wrench-system'/> -->
+    <!-- <plugin name='gz::sim::systems::NavSat' filename='gz-sim-navsat-system'/> -->
+    <plugin name='gz::sim::systems::Sensors' filename='gz-sim-sensors-system'>
+      <render_engine>ogre2</render_engine>
+    </plugin>
+    <!-- 3D scene -->
+    <plugin filename="MinimalScene" name="3D View">
+      <gz-gui>
+        <title>3D View</title>
+        <property type="bool" key="showTitleBar">false</property>
+        <property type="string" key="state">docked</property>
+      </gz-gui>
+      <engine>ogre2</engine>
+      <scene>scene</scene>
+      <ambient_light>0.4 0.4 0.4 1.0</ambient_light>
+      <background_color>0.7 0.7 0.7 1.0</background_color>
+      <camera_pose>-6 0 6 0 0.5 0</camera_pose>
+      <camera_clip>
+        <near>0.25</near>
+        <far>25000</far>
+      </camera_clip>
+    </plugin>
+    <!-- Scene Manager -->
+    <plugin filename="GzSceneManager" name="Scene Manager">
+      <gz-gui>
+        <property key="resizable" type="bool">true</property>
+        <property key="width" type="double">5</property>
+        <property key="height" type="double">5</property>
+        <property key="state" type="string">floating</property>
+        <property key="showTitleBar" type="bool">true</property>
+      </gz-gui>
+    </plugin>
+    <!-- World control -->
+    <plugin filename="WorldControl" name="World control">
+      <gz-gui>
+        <title>World control</title>
+        <property type="bool" key="showTitleBar">true</property>
+        <property type="bool" key="resizable">true</property>
+        <property type="double" key="height">72</property>
+        <property type="double" key="width">121</property>
+        <property type="double" key="z">1</property>
+        <property type="string" key="state">floating</property>
+        <anchors target="3D View">
+        <line own="left" target="left"/>
+        <line own="bottom" target="bottom"/>
+        </anchors>
+      </gz-gui>
+      <play_pause>true</play_pause>
+      <step>true</step>
+      <start_paused>true</start_paused>
+      <service>/world/world_demo/control</service>
+      <stats_topic>/world/world_demo/stats</stats_topic>
+    </plugin>
+  </xacro:macro>
 </sdf>

File: tmc_wrs_gazebo_worlds/worlds/wrs2020.world.xacro (robot description, xacro)
@@ -1,3 +1,3 @@
-<?xml version="1.0" ?>
+<?xml version="1.0" encoding="UTF-8" ?>
 <!--
 Copyright (c) 2017, Toyota Motor Corporation
@@ -25,10 +25,17 @@
 POSSIBILITY OF SUCH DAMAGE.
 -->
-<sdf version='1.6' xmlns:xacro="http://www.ros.org/wiki/xacro">
+<sdf version='1.8' xmlns:xacro="http://www.ros.org/wiki/xacro">
+  <xacro:include filename="$(find tmc_wrs_gz_worlds)/worlds/include/physics.xacro" />
   <xacro:arg name="fast_physics" default="true" />
   <xacro:arg name="highrtf" default="false" />
+  <xacro:arg name="trofast_knob" default="true" />
   <world name='default'>
+    <!-- Physics -->
+    <xacro:physics fast_physics="$(arg fast_physics)" highrtf="$(arg highrtf)" />
+    <!-- Sun light -->
     <light name='sun' type='directional'>
-      <cast_shadows>1</cast_shadows>
+      <xacro:if value="$(arg fast_physics)">
+        <cast_shadows>false</cast_shadows>
+      </xacro:if>
       <pose frame=''>0 0 10 0 -0 0</pose>
       <diffuse>0.8 0.8 0.8 1</diffuse>
@@ -42,13 +49,7 @@
       <direction>-0.5 0.1 -0.9</direction>
     </light>
+    <!-- Gravity -->
     <gravity>0 0 -9.8</gravity>
-    <xacro:include filename="include/physics.xacro" />
-    <scene>
-      <ambient>0.4 0.4 0.4 1</ambient>
-      <background>0.7 0.7 0.7 1</background>
-      <xacro:if value="$(arg fast_physics)">
-        <shadows>false</shadows>
-      </xacro:if>
-    </scene>
+    <!-- Include ground plane -->
     <include>
       <name>wrc_ground_plane</name>
@@ -155,16 +156,16 @@
       <pose frame=''>-2.7 0.1 0.4 0 -0 0</pose>
     </include>
-    <include>
+    <!-- <include>
       <name>person_standing</name>
       <static>1</static>
       <uri>model://person_standing</uri>
       <pose frame=''>0.7 1.5 0 0 -0 0</pose>
-    </include>
-    <include>
+    </include> -->
+    <!-- <include>
       <name>person_standing_0</name>
       <static>1</static>
       <uri>model://person_standing</uri>
       <pose frame=''>1.8 1.5 0 0 -0 0</pose>
-    </include>
+    </include> -->
   </world>
 </sdf>

Commit message: [FIX] unsupported conditional

File: tmc_wrs_gazebo_worlds/worlds/include/physics.xacro (robot description, xacro)
@@ -26,18 +26,20 @@
 -->
 <sdf version="1.8" xmlns:xacro="http://www.ros.org/wiki/xacro">
-  <xacro:macro name="physics" params="fast_physics:=true highrtf:=false" >
-    <physics name="1ms" type="ignored">
-      <xacro:if value="$(arg fast_physics)">
-        <xacro:unless value="$(arg highrtf)">
+  <xacro:macro name="physics" params="fast_physics:=true highrtf:=false">
+    <physics name="3ms" type="ignored">
+      <!-- <xacro:if value="$(eval fast_physics)">
+        <xacro:unless value="$(eval highrtf)">
           <real_time_update_rate>333.0</real_time_update_rate>
         </xacro:unless>
-        <xacro:if value="$(arg highrtf)">
+        <xacro:if value="$(eval highrtf)">
           <real_time_update_rate>0</real_time_update_rate>
         </xacro:if>
         <max_step_size>0.003</max_step_size>
       </xacro:if>
-      <xacro:if value="$(arg highrtf)">
+      <xacro:if value="$(eval highrtf)">
         <real_time_update_rate>0</real_time_update_rate>
-      </xacro:if>
+      </xacro:if> -->
+      <real_time_update_rate>333.0</real_time_update_rate>
+      <max_step_size>0.003</max_step_size>
     </physics>
     <plugin name='gz::sim::systems::Physics' filename='gz-sim-physics-system'/>

File: tmc_wrs_gazebo_worlds/worlds/wrs2020.world.xacro (robot description, xacro)
@@ -25,5 +25,5 @@
 POSSIBILITY OF SUCH DAMAGE.
 -->
-<sdf version='1.8' xmlns:xacro="http://www.ros.org/wiki/xacro">
+<sdf version='1.8' xmlns:xacro="http://ros.org/wiki/xacro">
   <xacro:include filename="$(find tmc_wrs_gz_worlds)/worlds/include/physics.xacro" />
   <xacro:arg name="fast_physics" default="true" />
@@ -35,8 +35,10 @@
     <!-- Sun light -->
     <light name='sun' type='directional'>
-      <xacro:if value="$(arg fast_physics)">
+      <!-- <xacro:if value="$(arg fast_physics)">
         <cast_shadows>false</cast_shadows>
-      </xacro:if>
-      <pose frame=''>0 0 10 0 -0 0</pose>
+      </xacro:if> -->
+      <!-- <cast_shadows>$(eval fast_physics ? 'false' : 'true')</cast_shadows> -->
+      <cast_shadows>true</cast_shadows>
+      <pose relative_to=''>0 0 10 0 -0 0</pose>
       <diffuse>0.8 0.8 0.8 1</diffuse>
       <specular>0.2 0.2 0.2 1</specular>
@@ -56,5 +58,5 @@
       <static>1</static>
       <uri>model://wrc_ground_plane</uri>
-      <pose frame=''>0 0 0 0 -0 0</pose>
+      <pose relative_to=''>0 0 0 0 -0 0</pose>
     </include>
     <include>
@@ -62,5 +64,5 @@
       <static>1</static>
       <uri>model://wrc_frame</uri>
-      <pose frame=''>0 0 0 0 -0 0</pose>
+      <pose relative_to=''>0 0 0 0 -0 0</pose>
     </include>
     <include>
@@ -68,5 +70,5 @@
       <uri>model://wrc_bookshelf</uri>
       <static>1</static>
-      <pose frame=''>2.7 -1 0 0 -0 -1.57</pose>
+      <pose relative_to=''>2.7 -1 0 0 -0 -1.57</pose>
     </include>
     <include>
@@ -74,5 +76,5 @@
       <static>1</static>
       <uri>model://wrc_bin_black</uri>
-      <pose frame=''>-2.7 -1.7 0 0 -0 0</pose>
+      <pose relative_to=''>-2.7 -1.7 0 0 -0 0</pose>
     </include>
     <include>
@@ -80,5 +82,5 @@
       <static>1</static>
       <uri>model://wrc_bin_green</uri>
-      <pose frame=''>-2.7 -1.2 0 0 -0 0</pose>
+      <pose relative_to=''>-2.7 -1.2 0 0 -0 0</pose>
     </include>
     <include>
@@ -86,35 +88,38 @@
       <static>1</static>
       <uri>model://wrc_stair_like_drawer</uri>
-      <pose frame=''>-2.7 1 0 0 -0 0</pose>
+      <pose relative_to=''>-2.7 1 0 0 -0 0</pose>
     </include>
     <include>
       <name>trofast_1</name>
-      <xacro:if value="$(arg trofast_knob)">
+      <!-- <xacro:if value="$(eval trofast_knob)">
         <uri>model://trofast_knob</uri>
       </xacro:if>
-      <xacro:unless value="$(arg trofast_knob)">
+      <xacro:unless value="$(eval trofast_knob)">
         <uri>model://trofast</uri>
-      </xacro:unless>
-      <pose frame=''>-2.7 0.67 0.1 0 -0 0</pose>
+      </xacro:unless> -->
+      <uri>model://trofast_knob</uri>
+      <pose relative_to=''>-2.7 0.67 0.1 0 -0 0</pose>
     </include>
     <include>
       <name>trofast_2</name>
-      <xacro:if value="$(arg trofast_knob)">
+      <!-- <xacro:if value="$(eval trofast_knob)">
         <uri>model://trofast_knob</uri>
       </xacro:if>
-      <xacro:unless value="$(arg trofast_knob)">
+      <xacro:unless value="$(eval trofast_knob)">
         <uri>model://trofast</uri>
-      </xacro:unless>
-      <pose frame=''>-2.7 1 0.1 0 -0 0</pose>
+      </xacro:unless> -->
+      <uri>model://trofast_knob</uri>
+      <pose relative_to=''>-2.7 1 0.1 0 -0 0</pose>
     </include>
     <include>
       <name>trofast_3</name>
-      <xacro:if value="$(arg trofast_knob)">
+      <!-- <xacro:if value="$(eval trofast_knob)">
         <uri>model://trofast_knob</uri>
       </xacro:if>
-      <xacro:unless value="$(arg trofast_knob)">
+      <xacro:unless value="$(eval trofast_knob)">
         <uri>model://trofast</uri>
-      </xacro:unless>
-      <pose frame=''>-2.7 1 0.36 0 -0 0</pose>
+      </xacro:unless> -->
+      <uri>model://trofast_knob</uri>
+      <pose relative_to=''>-2.7 1 0.36 0 -0 0</pose>
     </include>
     <include>
@@ -122,5 +127,5 @@
       <static>1</static>
       <uri>model://wrc_tall_table</uri>
-      <pose frame=''>-0.3 1.2 0 0 -0 0</pose>
+      <pose relative_to=''>-0.3 1.2 0 0 -0 0</pose>
     </include>
     <include>
@@ -128,5 +133,5 @@
       <static>1</static>
       <uri>model://wrc_long_table</uri>
-      <pose frame=''>-0.3 0.2 0 0 -0 1.57</pose>
+      <pose relative_to=''>-0.3 0.2 0 0 -0 1.57</pose>
     </include>
     <include>
@@ -134,25 +139,25 @@
       <static>1</static>
       <uri>model://wrc_long_table</uri>
-      <pose frame=''>-2.7 -0.3 0 0 -0 1.57</pose>
+      <pose relative_to=''>-2.7 -0.3 0 0 -0 1.57</pose>
     </include>
     <include>
       <name>wrc_tray_1</name>
       <uri>model://wrc_tray</uri>
-      <pose frame=''>-2.7 -0.75 0.4 0 -0 1.57</pose>
+      <pose relative_to=''>-2.7 -0.75 0.4 0 -0 1.57</pose>
     </include>
     <include>
       <name>wrc_tray_2</name>
       <uri>model://wrc_tray</uri>
-      <pose frame=''>-2.7 -0.45 0.4 0 -0 1.57</pose>
+      <pose relative_to=''>-2.7 -0.45 0.4 0 -0 1.57</pose>
     </include>
     <include>
       <name>wrc_container_a</name>
       <uri>model://wrc_container_a</uri>
-      <pose frame=''>-2.7 -0.2 0.4 0 -0 0</pose>
+      <pose relative_to=''>-2.7 -0.2 0.4 0 -0 0</pose>
     </include>
     <include>
       <name>wrc_container_b</name>
       <uri>model://wrc_container_b</uri>
-      <pose frame=''>-2.7 0.1 0.4 0 -0 0</pose>
+      <pose relative_to=''>-2.7 0.1 0.4 0 -0 0</pose>
     </include>
     <!-- <include>
@@ -160,5 +165,5 @@
       <static>1</static>
       <uri>model://person_standing</uri>
-      <pose frame=''>0.7 1.5 0 0 -0 0</pose>
+      <pose relative_to=''>0.7 1.5 0 0 -0 0</pose>
     </include> -->
     <!-- <include>
@@ -166,5 +171,5 @@
       <static>1</static>
       <uri>model://person_standing</uri>
-      <pose frame=''>1.8 1.5 0 0 -0 0</pose>
+      <pose relative_to=''>1.8 1.5 0 0 -0 0</pose>
     </include> -->
   </world>
